File: engine-controller/thermocouple.kicad_sch (KiCad schematic)
At the start: 6 parts, among them IC301 MAX31856MUD+

Commit message: initial layout
Parts:
- IC301: footprint SOP65P640X110-14N -> SamacSys_Parts:SOP65P640X110-14N
Changed lines of the file:
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@@
       (effects (font (size 1.27 1.27)))
     )
-    (property "Footprint" "SOP65P640X110-14N" (at 158.75 164.77 0)
+    (property "Footprint" "SamacSys_Parts:SOP65P640X110-14N" (at 158.75 164.77 0)
       (effects (font (size 1.27 1.27)) (justify left top) hide)
     )
